File: hardware/Transmitter board/proejtc.kicad_pcb (KiCad board)
At the start: 2 copper layers, 31.5 x 24.5 mm, 4 parts, among them U1 PAM8403D, U2 MAX4466EXK_T

Commit message: Add files via upload
Parts:
- removed U2: MAX4466EXK_T, digikey-footprints:SOT-353
- added J1: Conn_01x03_Pin, Connector_PinSocket_2.54mm:PinSocket_1x03_P2.54mm_Horizontal, F.Cu at (152.9, 100.5)
Connections:
- R1 pad 2: Net-(LD1-A) -> Net-(LD1-C)
- U1 pad 1: Net-(LD1-C) -> Net-(LD1-A)
- U1 pad 12: +5V -> unconnected-(U1-~{SHDN}-Pad12)
- U1 pad 5: +5V -> unconnected-(U1-~{MUTE}-Pad5)
Routing:
- net Net-(J1-Pin_1): track 41.1 -> 14.9 mm
- net Net-(LD1-A): track 5.25 -> 6.26 mm
- net Net-(LD1-C): track 6.43 -> 7.33 mm
- net +5V: track 19.1 -> 19.2 mm, vias 0 -> 2
